File: nes_memories.kicad_sch (KiCad schematic)
At the start: 6 parts, among them U5 IS61C5128AL-10TLI, U6 IS61C5128AL-10TLI

Commit message: Create project-local libraries
Signed-off-by: Chris Frantz <frantzcj@gmail.com>
Parts:
- C1, C3, C4, C5: symbol Device:C -> Library:C
- U5, U6: symbol Memory_RAM:IS61C5128AL-10TLI -> Library:IS61C5128AL-10TLI
Changed lines of the file:
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@@
 	)
 	(symbol
-		(lib_id "Device:C")
+		(lib_id "Library:C")
 		(at 194.31 29.21 90)
 		(unit 1)
@@
 	)
 	(symbol
-		(lib_id "Memory_RAM:IS61C5128AL-10TLI")
+		(lib_id "Library:IS61C5128AL-10TLI")
 		(at 190.5 81.28 0)
 		(unit 1)
@@
 	)
 	(symbol
-		(lib_id "power:GND")
+		(lib_id "Library:GND")
 		(at 190.5 114.3 0)
 		(unit 1)
@@
 	)
 	(symbol
-		(lib_id "power:GND")
+		(lib_id "Library:GND")
 		(at 63.5 114.3 0)
 		(unit 1)
@@
 	)
 	(symbol
-		(lib_id "Device:C")
+		(lib_id "Library:C")
 		(at 194.31 36.83 90)
 		(unit 1)
@@
 	)
 	(symbol
-		(lib_id "power:VCC")
+		(lib_id "Library:VCC")
 		(at 190.5 27.94 0)
 		(unit 1)
@@
 	)
 	(symbol
-		(lib_id "Device:C")
+		(lib_id "Library:C")
 		(at 67.31 29.21 90)
 		(unit 1)
@@
 	)
 	(symbol
-		(lib_id "Memory_RAM:IS61C5128AL-10TLI")
+		(lib_id "Library:IS61C5128AL-10TLI")
 		(at 63.5 81.28 0)
 		(unit 1)
@@
 	)
 	(symbol
-		(lib_id "power:VCC")
+		(lib_id "Library:VCC")
 		(at 63.5 27.94 0)
 		(unit 1)
@@
 	)
 	(symbol
-		(lib_id "power:GND")
+		(lib_id "Library:GND")
 		(at 198.12 36.83 0)
 		(unit 1)
@@
 	)
 	(symbol
-		(lib_id "Device:C")
+		(lib_id "Library:C")
 		(at 67.31 36.83 90)
 		(unit 1)
@@
 	)
 	(symbol
-		(lib_id "power:GND")
+		(lib_id "Library:GND")
 		(at 71.12 36.83 0)
 		(unit 1)
