File: nes_5v.kicad_sch (KiCad schematic)
At the start: 2 parts, among them CN2 NES Card Edge, J1 NES 5v TP

Commit message: Create project-local libraries
Signed-off-by: Chris Frantz <frantzcj@gmail.com>
Parts:
- CN2: symbol Personal_Library:NES_Card_Edge -> Library:NES_Card_Edge
- J1: symbol Connector_Generic:Conn_02x36_Odd_Even -> Library:Conn_02x36_Odd_Even
Changed lines of the file:
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@@
 	)
 	(symbol
-		(lib_id "power:GND")
+		(lib_id "Library:GND")
 		(at 83.82 140.97 0)
 		(unit 1)
@@
 	)
 	(symbol
-		(lib_id "power:VCC")
+		(lib_id "Library:VCC")
 		(at 266.7 54.61 0)
 		(unit 1)
@@
 	)
 	(symbol
-		(lib_id "power:GND")
+		(lib_id "Library:GND")
 		(at 213.36 54.61 0)
 		(unit 1)
@@
 	)
 	(symbol
-		(lib_id "Personal_Library:NES_Card_Edge")
+		(lib_id "Library:NES_Card_Edge")
 		(at 114.3 97.79 0)
 		(unit 1)
@@
 	)
 	(symbol
-		(lib_id "power:VCC")
+		(lib_id "Library:VCC")
 		(at 83.82 46.99 0)
 		(unit 1)
@@
 	)
 	(symbol
-		(lib_id "Connector_Generic:Conn_02x36_Odd_Even")
+		(lib_id "Library:Conn_02x36_Odd_Even")
 		(at 243.84 97.79 0)
 		(unit 1)
@@
 	)
 	(symbol
-		(lib_id "power:GND")
+		(lib_id "Library:GND")
 		(at 132.08 39.37 0)
 		(unit 1)
@@
 	)
 	(symbol
-		(lib_id "power:GND")
+		(lib_id "Library:GND")
 		(at 266.7 143.51 0)
 		(unit 1)
