File: nes_power.kicad_sch (KiCad schematic)
At the start: 9 parts, among them J3 NES PWR, U7 LM3671-3.3, U8 LM3671-1.2

Commit message: Create project-local libraries
Signed-off-by: Chris Frantz <frantzcj@gmail.com>
Parts:
- C15, C16, C17, C18: symbol Device:C -> Library:C
- J3: symbol Connector:Conn_01x02_Pin -> Library:Conn_01x02_Pin
- L1, L2: symbol Device:L -> Library:L
- U7, U8: symbol Regulator_Switching:LM3670MF -> Library:LM3670MF
Changed lines of the file:
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@@
 	)
 	(symbol
-		(lib_id "Connector:Conn_01x02_Pin")
+		(lib_id "Library:Conn_01x02_Pin")
 		(at 40.64 48.26 0)
 		(unit 1)
@@
 	)
 	(symbol
-		(lib_id "power:VCC")
+		(lib_id "Library:VCC")
 		(at 45.72 39.37 0)
 		(unit 1)
@@
 	)
 	(symbol
-		(lib_id "power:VCC")
+		(lib_id "Library:VCC")
 		(at 110.49 81.28 0)
 		(unit 1)
@@
 	)
 	(symbol
-		(lib_id "Device:C")
+		(lib_id "Library:C")
 		(at 60.96 57.15 0)
 		(unit 1)
@@
 	)
 	(symbol
-		(lib_id "Device:L")
+		(lib_id "Library:L")
 		(at 88.9 50.8 90)
 		(unit 1)
@@
 	)
 	(symbol
-		(lib_id "Device:L")
+		(lib_id "Library:L")
 		(at 88.9 81.28 90)
 		(unit 1)
@@
 	)
 	(symbol
-		(lib_id "power:VCC")
+		(lib_id "Library:VCC")
 		(at 110.49 50.8 0)
 		(unit 1)
@@
 	)
 	(symbol
-		(lib_id "Regulator_Switching:LM3670MF")
+		(lib_id "Library:LM3670MF")
 		(at 77.47 53.34 0)
 		(unit 1)
@@
 	)
 	(symbol
-		(lib_id "Device:C")
+		(lib_id "Library:C")
 		(at 60.96 87.63 0)
 		(unit 1)
@@
 	)
 	(symbol
-		(lib_id "Regulator_Switching:LM3670MF")
+		(lib_id "Library:LM3670MF")
 		(at 77.47 83.82 0)
 		(unit 1)
@@
 	)
 	(symbol
-		(lib_id "power:GND")
+		(lib_id "Library:GND")
 		(at 77.47 93.98 0)
 		(unit 1)
@@
 	)
 	(symbol
-		(lib_id "Device:C")
+		(lib_id "Library:C")
 		(at 102.87 87.63 0)
 		(unit 1)
@@
 	)
 	(symbol
-		(lib_id "Device:C")
+		(lib_id "Library:C")
 		(at 102.87 57.15 0)
 		(unit 1)
@@
 	)
 	(symbol
-		(lib_id "power:GND")
+		(lib_id "Library:GND")
 		(at 77.47 63.5 0)
 		(unit 1)

Commit message: Update footprints and schematic.
1. Update teh HX8K eval board footprint to group power & grounds.
2. Re-arrange the level shifter section to try to get a better "straight
   through" layout.

Signed-off-by: Chris Frantz <frantzcj@gmail.com>
Parts:
- U7, U8: footprint Package_TO_SOT_SMD:SOT-23-5 -> Package_TO_SOT_SMD:TSOT-23-5
Changed lines of the file:
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@@
 			)
 		)
-		(property "Footprint" "Package_TO_SOT_SMD:SOT-23-5"
+		(property "Footprint" "Package_TO_SOT_SMD:TSOT-23-5"
 			(at 78.74 59.69 0)
 			(effects
@@
 			)
 		)
-		(property "Footprint" "Package_TO_SOT_SMD:SOT-23-5"
+		(property "Footprint" "Package_TO_SOT_SMD:TSOT-23-5"
 			(at 78.74 90.17 0)
 			(effects
